Commit message: Added xacro macro argument to laser mount to choose min and max laser angle

File: multi_warthog_description/urdf/accessories.urdf.xacro (robot description, xacro)
@@ -12,5 +12,7 @@
   <xacro:if value="$(optenv WARTHOG_LASER 0)">
     <sick_lms1xx_mount prefix="$(optenv WARTHOG_LASER_MOUNT front)"
-                       topic="$(optenv WARTHOG_LASER_TOPIC front/scan)"/>
+                       topic="$(optenv WARTHOG_LASER_TOPIC front/scan)"
+                       min_angle="-1.7"
+                       max_angle="1.7" />
     <joint name="$(optenv WARTHOG_LASER_MOUNT front)_laser_mount_joint" type="fixed">
       <origin xyz="$(optenv WARTHOG_LASER_OFFSET 0.77 0 0.15)"
@@ -23,5 +25,7 @@
   <xacro:if value="$(optenv WARTHOG_LASER 0)">
     <sick_lms1xx_mount prefix="$(optenv WARTHOG_LASER_MOUNT back)"
-                       topic="$(optenv WARTHOG_LASER_TOPIC back/scan)"/>
+                       topic="$(optenv WARTHOG_LASER_TOPIC back/scan)"
+                       min_angle="-1.7"
+                       max_angle="1.7" />
     <joint name="$(optenv WARTHOG_LASER_MOUNT back)_laser_mount_joint" type="fixed">
       <origin xyz="$(optenv WARTHOG_LASER_OFFSET -0.77 0 0.15)"

File: multi_warthog_description/urdf/accessories/sick_lms1xx_mount.urdf.xacro (robot description, xacro)
@@ -27,6 +27,6 @@
 <robot xmlns:xacro="http://www.ros.org/wiki/xacro">
   <xacro:include filename="$(find lms1xx)/urdf/sick_lms1xx.urdf.xacro" />
-  <xacro:macro name="sick_lms1xx_mount" params="prefix topic">
-    <sick_lms1xx frame="${prefix}_laser" topic="${topic}" robot_namespace="$(arg namespace)" />
+  <xacro:macro name="sick_lms1xx_mount" params="prefix topic min_angle max_angle">
+    <sick_lms1xx frame="${prefix}_laser" topic="${topic}" robot_namespace="$(arg namespace)" min_angle="${min_angle}" max_angle="${max_angle}"/>
     <link name="${prefix}_laser_mount">
       <visual>

File: multi_warthog_description/urdf/warthog.urdf.xacro (robot description, xacro)
@@ -47,5 +47,5 @@
         <origin xyz="0 0 0" rpy="0 0 ${PI/2}"/>
         <geometry>
-          <mesh filename="package://warthog_description/meshes/wheel.stl" />
+          <mesh filename="package://multi_warthog_description/meshes/wheel.stl" />
         </geometry>
         <material name="dark_grey" />
@@ -89,5 +89,5 @@
         <origin xyz="0 0 0" rpy="0 0 0"/>
         <geometry>
-          <mesh filename="package://warthog_description/meshes/tracks.dae" />
+          <mesh filename="package://multi_warthog_description/meshes/tracks.dae" />
         </geometry>
         <material name="dark_grey" />
@@ -96,5 +96,5 @@
         <origin xyz="0 0 0" rpy="0 0 0"/>
         <geometry>
-          <mesh filename="package://warthog_description/meshes/tracks_collision.stl" />
+          <mesh filename="package://multi_warthog_description/meshes/tracks_collision.stl" />
         </geometry>
       </collision>
@@ -171,5 +171,5 @@
         <origin xyz="0 0 0" rpy="0 0 ${side*PI/2}"/>
         <geometry>
-          <mesh filename="package://warthog_description/meshes/rocker.stl" />
+          <mesh filename="package://multi_warthog_description/meshes/rocker.stl" />
         </geometry>
         <material name="black"><color rgba="0.15 0.15 0.15 1.0" /></material>
@@ -178,5 +178,5 @@
         <origin xyz="0 0 0" rpy="0 0 ${side*PI/2}"/>
         <geometry>
-          <mesh filename="package://warthog_description/meshes/fenders.stl" />
+          <mesh filename="package://multi_warthog_description/meshes/fenders.stl" />
         </geometry>
         <material name="yellow"><color rgba="0.95 0.816 0.082 1.0" /></material>
@@ -185,5 +185,5 @@
         <origin xyz="0 ${side*-0.0244} 0" rpy="0 0 0"/>
         <geometry>
-          <mesh filename="package://warthog_description/meshes/light.stl" />
+          <mesh filename="package://multi_warthog_description/meshes/light.stl" />
         </geometry>
         <material name="white"><color rgba="0.9 0.9 0.9 1.0" /></material>
@@ -192,5 +192,5 @@
         <origin xyz="0 ${side*-0.0244} 0" rpy="0 0 ${side*PI}"/>
         <geometry>
-          <mesh filename="package://warthog_description/meshes/light.stl" />
+          <mesh filename="package://multi_warthog_description/meshes/light.stl" />
         </geometry>
         <material name="red"><color rgba="0.9 0.0 0.0 1.0" /></material>
@@ -199,5 +199,5 @@
         <origin xyz="0 0 0" rpy="0 0 ${side*PI/2}"/>
         <geometry>
-          <mesh filename="package://warthog_description/meshes/fenders.stl" />
+          <mesh filename="package://multi_warthog_description/meshes/fenders.stl" />
         </geometry>
       </collision>
@@ -234,5 +234,5 @@
       <origin xyz="0 0 0" rpy="0 0 0"/>
       <geometry>
-        <mesh filename="package://warthog_description/meshes/chassis.stl" />
+        <mesh filename="package://multi_warthog_description/meshes/chassis.stl" />
       </geometry>
       <material name="black"><color rgba="0.15 0.15 0.15 1.0" /></material>
@@ -241,5 +241,5 @@
       <origin xyz="0 0 0" rpy="0 0 0"/>
       <geometry>
-        <mesh filename="package://warthog_description/meshes/e-stop.stl" />
+        <mesh filename="package://multi_warthog_description/meshes/e-stop.stl" />
       </geometry>
       <material name="red"><color rgba="0.9 0.0 0.0 1.0" /></material>
@@ -248,5 +248,5 @@
       <origin xyz="0 0 0" rpy="0 0 0"/>
       <geometry>
-        <mesh filename="package://warthog_description/meshes/chassis-collision.stl" />
+        <mesh filename="package://multi_warthog_description/meshes/chassis-collision.stl" />
       </geometry>
     </collision>
@@ -263,5 +263,5 @@
       <origin xyz="0 0 0" rpy="0 0 0"/>
       <geometry>
-        <mesh filename="package://warthog_description/meshes/diff-link.stl" />
+        <mesh filename="package://multi_warthog_description/meshes/diff-link.stl" />
       </geometry>
       <material name="light_grey" />
@@ -270,5 +270,5 @@
       <origin xyz="0 0 0" rpy="0 0 0"/>
       <geometry>
-        <mesh filename="package://warthog_description/meshes/susp-link.stl" />
+        <mesh filename="package://multi_warthog_description/meshes/susp-link.stl" />
       </geometry>
       <material name="light_grey" />
@@ -277,5 +277,5 @@
       <origin xyz="0 0 0" rpy="0 0 0"/>
       <geometry>
-        <mesh filename="package://warthog_description/meshes/susp-link.stl" />
+        <mesh filename="package://multi_warthog_description/meshes/susp-link.stl" />
       </geometry>
       <material name="light_grey" />
@@ -294,9 +294,9 @@
   </joint>
   <!-- Bring in simulation data for Gazebo. -->
-  <xacro:include filename="$(find warthog_description)/urdf/warthog.gazebo" />
+  <xacro:include filename="$(find multi_warthog_description)/urdf/warthog.gazebo" />
   <!-- Optional standard accessories, including their simulation data. The rendering
        of these into the final description is controlled by optenv variables, which
        default each one to off.-->
-  <xacro:include filename="$(find warthog_description)/urdf/accessories.urdf.xacro" />
+  <xacro:include filename="$(find multi_warthog_description)/urdf/accessories.urdf.xacro" />
   <!-- Optional custom includes. -->
   <xacro:include filename="$(optenv WARTHOG_URDF_EXTRAS empty.urdf)" />
