Commit message: Update for solarfarm

File: multi_warthog_description/urdf/accessories/sick_lms1xx_mount.urdf.xacro (robot description, xacro)
@@ -34,5 +34,5 @@
         <geometry>
           <!-- Origin of this mesh is the base of the bracket. -->
-          <mesh filename="package://warthog_description/meshes/sick-lms1xx-bracket.stl" />
+          <mesh filename="package://multi_warthog_description/meshes/sick-lms1xx-bracket.stl" />
         </geometry>
         <material name="dark_grey" />

File: multi_warthog_description/urdf/accessories/warthog_arm_mount.urdf.xacro (robot description, xacro)
@@ -6,5 +6,5 @@
         <origin xyz="0 0 0" rpy="0 0 0"/>
         <geometry>
-          <mesh filename="package://warthog_description/meshes/arm-mount-plate.stl" />
+          <mesh filename="package://multi_warthog_description/meshes/arm-mount-plate.stl" />
         </geometry>
         <material name="light_grey"/>
@@ -13,5 +13,5 @@
         <origin xyz="0 0 0" rpy="0 0 0"/>
         <geometry>
-          <mesh filename="package://warthog_description/meshes/arm-mount-plate.stl" />
+          <mesh filename="package://multi_warthog_description/meshes/arm-mount-plate.stl" />
         </geometry>
       </collision>

File: multi_warthog_description/urdf/accessories/warthog_bulkhead.urdf.xacro (robot description, xacro)
@@ -6,5 +6,5 @@
         <origin xyz="0 0 0" rpy="0 0 0"/>
         <geometry>
-          <mesh filename="package://warthog_description/meshes/bulkhead.stl" />
+          <mesh filename="package://multi_warthog_description/meshes/bulkhead.stl" />
         </geometry>
         <material name="black"><color rgba="0.15 0.15 0.15 1.0" /></material>
@@ -13,5 +13,5 @@
         <origin xyz="0 0 0" rpy="0 0 0"/>
         <geometry>
-          <mesh filename="package://warthog_description/meshes/bulkhead-collision.stl" />
+          <mesh filename="package://multi_warthog_description/meshes/bulkhead-collision.stl" />
         </geometry>
       </collision>

File: multi_warthog_description/urdf/warthog.urdf.xacro (robot description, xacro)
@@ -66,6 +66,6 @@
     <gazebo reference="${prefix}_${side}_wheel_link">
       <selfCollide>false</selfCollide>
-      <mu1>0.5</mu1>
-      <mu2>0.5</mu2>
+      <mu1>1</mu1>
+      <mu2>1</mu2>
       <kp value="10000000.0" />
       <kd value="1.0" />
